File: luncheonmeat.sch (KiCad schematic (older format))
At the start: 37 parts, among them J1 USB_B_Micro, Q1 Q_PMOS_DGS, Q2 Q_PMOS_DGS, Q3 Q_PMOS_DGS, SW1 SW_Push, SW10 9, SW11 6, SW12 3, SW13 #, SW2 7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

Commit message: progress
Parts:
- added C10, C8, C9: 100n, Capacitor_SMD:C_0603_1608Metric_Pad1.05x0.95mm_HandSolder, symbol Device:C
- added C11: 4u7, Capacitor_SMD:C_0603_1608Metric_Pad1.05x0.95mm_HandSolder, symbol Device:C
- added D1: LED, Diode_SMD:D_0603_1608Metric_Pad1.05x0.95mm_HandSolder, symbol Device:LED
- added J2: Conn_02x03_Odd_Even, Connector_PinHeader_2.54mm:PinHeader_2x03_P2.54mm_Vertical, symbol Connector_Generic:Conn_02x03_Odd_Even
- added R10, R11, R12, R13, R14, R15, R16, R7, R8, R9: 300R, Resistor_SMD:R_0603_1608Metric_Pad1.05x0.95mm_HandSolder, symbol Device:R
- J1: footprint Connector_USB:USB_Micro-B_Molex-105017-0001 -> Connector_USB:USB_Micro-B_Wuerth_629105150521_CircularHoles
- R1: value R -> 100k
- R2, R3, R4: footprint Resistor_SMD:R_0201_0603Metric -> Resistor_SMD:R_0603_1608Metric_Pad1.05x0.95mm_HandSolder
- SW10: value 9 -> 7
- SW11: value 6 -> 4
- SW12: value 3 -> 1
- SW13: value # -> *
- SW2: value 7 -> 9
- SW3: value 4 -> 6
- SW4: value 1 -> 3
- SW5: value * -> #
- Y1: value Crystal -> 16MHz; footprint Crystal:Crystal_HC49-U_Vertical -> Crystal:Crystal_HC49-4H_Vertical; symbol Device:Crystal -> Device:Crystal_Small
Connections:
- net +5V: now also U1.18 (AVCC), U1.20 (AREF), U1.4 (VCC), C10.1, C11.1, C8.1, C9.1, D1.2 (A), J2.2 (Pin_2)
- net COL_0: now also U1.12 (PB0); no longer U1.3 (PE0)
- net COL_1: now also U1.13 (PB1); no longer U1.6 (PE1)
- net COL_2: now also U1.14 (PB2); no longer U1.19 (PE2)
- net Earth: now also U1.21 (GND), U1.5 (GND), C10.2, C11.2, C8.2, C9.2, J2.6 (Pin_6), R16.2
- net ROW_0: now also U1.3 (PE0); no longer U1.12 (PB0)
- net ROW_1: now also U1.6 (PE1); no longer U1.13 (PB1)
- net ROW_2: now also U1.19 (PE2); no longer U1.14 (PB2)
- net ROW_3: now also U1.22 (PE3); no longer U1.15 (PB3)
- net SEG_A: now also R7.1; no longer U1.30 (PD0)
- net SEG_B: now also R8.1; no longer U1.31 (PD1)
- net SEG_C: now also R9.1; no longer U1.32 (PD2)
- net SEG_D: now also R10.1; no longer U1.1 (PD3)
- net SEG_E: now also R11.1; no longer U1.2 (PD4)
- net SEG_F: now also R12.1; no longer U1.9 (PD5)
- net SEG_G: now also R13.1; no longer U1.10 (PD6)
- net SEG_RDP: now also R14.1; no longer U1.11 (PD7)
- net SEG_SEL_0: now also U1.2 (PD4); no longer U1.23 (PC0)
- net SEG_SEL_1: now also U1.9 (PD5); no longer U1.24 (PC1)
- net SEG_SEL_2: now also U1.10 (PD6); no longer U1.25 (PC2)
- net MISO: now reaches U1.16 (PB4)
- net MISO: now also J2.1 (Pin_1)
- net SCK: now reaches U1.17 (PB5)
- net SCK: now also J2.3 (Pin_3)
- net at U1.26 (PC3): now also R10.2
- net at U1.27 (PC4): now also R11.2
- net at U1.28 (PC5): now also R12.2
- net at C1.2, R1.2, SW1.1: now also R15.1; no longer U1.29 (~RESET~/PC6)
- net TX: now reaches U5.1 (TXD)
- net TX: now also U1.31 (PD1)
- net RX: now reaches U5.4 (RXD)
- net RX: now also U1.30 (PD0)
- new net: R14.2, U1.1 (PD3)
- new net: R7.2, U1.23 (PC0)
- new net: R8.2, U1.24 (PC1)
- new net: R9.2, U1.25 (PC2)
- new net: R13.2, U1.32 (PD2)
- new net: D1.1 (K), R16.1
- new net MOSI: J2.4 (Pin_4), U1.15 (PB3)
- new net RESET: J2.5 (Pin_5), R15.2, U1.29 (~RESET~/PC6)
Other:
- moved on the sheet: C1, C2, C3, C4, C5, C6, C7, J1, L1, Q1, Q2, Q3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

Commit message: progress
Parts:
- SW1: footprint Button_Switch_THT:SW_PUSH_6mm -> Connector_PinHeader_2.54mm:PinHeader_1x02_P2.54mm_Vertical
Other:
- moved on the sheet: C10, C11, C8, C9, D1, R16
Changed lines of the file:
@@
 F 0 "SW1" V 7454 5298 50  0000 L CNN
 F 1 "SW_Push" V 7545 5298 50  0000 L CNN
-F 2 "Button_Switch_THT:SW_PUSH_6mm" H 7500 5350 50  0001 C CNN
+F 2 "Connector_PinHeader_2.54mm:PinHeader_1x02_P2.54mm_Vertical" H 7500 5350 50  0001 C CNN
 F 3 "~" H 7500 5350 50  0001 C CNN
 	1    7500 5150
@@
 L power:+5V #PWR0108
 U 1 1 5FC5EF24
-P 2500 4350
-F 0 "#PWR0108" H 2500 4200 50  0001 C CNN
-F 1 "+5V" H 2515 4523 50  0000 C CNN
-F 2 "" H 2500 4350 50  0001 C CNN
-F 3 "" H 2500 4350 50  0001 C CNN
-	1    2500 4350
+P 2500 4450
+F 0 "#PWR0108" H 2500 4300 50  0001 C CNN
+F 1 "+5V" H 2515 4623 50  0000 C CNN
+F 2 "" H 2500 4450 50  0001 C CNN
+F 3 "" H 2500 4450 50  0001 C CNN
+	1    2500 4450
 	1    0    0    -1
 $EndComp
@@
 	2450 4550 2500 4550
 Wire Wire Line
-	2500 4550 2500 4350
+	2500 4550 2500 4450
 Wire Wire Line
 	2500 4550 4450 4550
@@
 L Device:C C8
 U 1 1 60C31B9F
-P 6450 5950
-F 0 "C8" H 6565 5996 50  0000 L CNN
-F 1 "100n" H 6565 5905 50  0000 L CNN
-F 2 "Capacitor_SMD:C_0603_1608Metric_Pad1.05x0.95mm_HandSolder" H 6488 5800 50  0001 C CNN
-F 3 "~" H 6450 5950 50  0001 C CNN
-	1    6450 5950
+P 6200 5850
+F 0 "C8" H 6315 5896 50  0000 L CNN
+F 1 "100n" H 6315 5805 50  0000 L CNN
+F 2 "Capacitor_SMD:C_0603_1608Metric_Pad1.05x0.95mm_HandSolder" H 6238 5700 50  0001 C CNN
+F 3 "~" H 6200 5850 50  0001 C CNN
+	1    6200 5850
 	1    0    0    -1
 $EndComp
@@
 L power:+5V #PWR02
 U 1 1 60C3BFA6
-P 6450 5700
-F 0 "#PWR02" H 6450 5550 50  0001 C CNN
-F 1 "+5V" H 6465 5873 50  0000 C CNN
-F 2 "" H 6450 5700 50  0001 C CNN
-F 3 "" H 6450 5700 50  0001 C CNN
-	1    6450 5700
+P 6200 5600
+F 0 "#PWR02" H 6200 5450 50  0001 C CNN
+F 1 "+5V" H 6215 5773 50  0000 C CNN
+F 2 "" H 6200 5600 50  0001 C CNN
+F 3 "" H 6200 5600 50  0001 C CNN
+	1    6200 5600
 	1    0    0    -1
 $EndComp
@@
 L Device:C C9
 U 1 1 60D62166
-P 6850 5950
-F 0 "C9" H 6965 5996 50  0000 L CNN
-F 1 "100n" H 6965 5905 50  0000 L CNN
-F 2 "Capacitor_SMD:C_0603_1608Metric_Pad1.05x0.95mm_HandSolder" H 6888 5800 50  0001 C CNN
-F 3 "~" H 6850 5950 50  0001 C CNN
-	1    6850 5950
+P 6600 5850
+F 0 "C9" H 6715 5896 50  0000 L CNN
+F 1 "100n" H 6715 5805 50  0000 L CNN
+F 2 "Capacitor_SMD:C_0603_1608Metric_Pad1.05x0.95mm_HandSolder" H 6638 5700 50  0001 C CNN
+F 3 "~" H 6600 5850 50  0001 C CNN
+	1    6600 5850
 	1    0    0    -1
 $EndComp
@@
 L Device:C C10
 U 1 1 60D62432
-P 7250 5950
-F 0 "C10" H 7365 5996 50  0000 L CNN
-F 1 "100n" H 7365 5905 50  0000 L CNN
-F 2 "Capacitor_SMD:C_0603_1608Metric_Pad1.05x0.95mm_HandSolder" H 7288 5800 50  0001 C CNN
-F 3 "~" H 7250 5950 50  0001 C CNN
-	1    7250 5950
+P 7000 5850
+F 0 "C10" H 7115 5896 50  0000 L CNN
+F 1 "100n" H 7115 5805 50  0000 L CNN
+F 2 "Capacitor_SMD:C_0603_1608Metric_Pad1.05x0.95mm_HandSolder" H 7038 5700 50  0001 C CNN
+F 3 "~" H 7000 5850 50  0001 C CNN
+	1    7000 5850
 	1    0    0    -1
 $EndComp
@@
 L power:Earth #PWR03
 U 1 1 60D63DB9
-P 6450 6200
-F 0 "#PWR03" H 6450 5950 50  0001 C CNN
-F 1 "Earth" H 6450 6050 50  0001 C CNN
-F 2 "" H 6450 6200 50  0001 C CNN
-F 3 "~" H 6450 6200 50  0001 C CNN
-	1    6450 6200
-	1    0    0    -1
-$EndComp
-Wire Wire Line
-	7250 5800 7250 5750
-Wire Wire Line
-	7250 5750 6850 5750
-Wire Wire Line
-	6850 5750 6850 5800
-Wire Wire Line
-	6850 5750 6450 5750
-Wire Wire Line
-	6450 5750 6450 5800
-Connection ~ 6850 5750
-Wire Wire Line
-	6450 5700 6450 5750
-Wire Wire Line
-	6850 6100 6850 6150
-Wire Wire Line
-	6450 6150 6450 6100
-Wire Wire Line
-	6450 6150 6850 6150
-Connection ~ 6850 6150
-Wire Wire Line
-	6450 6150 6450 6200
-Wire Wire Line
-	7250 6100 7250 6150
-Wire Wire Line
-	7250 6150 6850 6150
+P 6200 6100
+F 0 "#PWR03" H 6200 5850 50  0001 C CNN
+F 1 "Earth" H 6200 5950 50  0001 C CNN
+F 2 "" H 6200 6100 50  0001 C CNN
+F 3 "~" H 6200 6100 50  0001 C CNN
+	1    6200 6100
+	1    0    0    -1
+$EndComp
+Wire Wire Line
+	7000 5700 7000 5650
+Wire Wire Line
+	7000 5650 6600 5650
+Wire Wire Line
+	6600 5650 6600 5700
+Wire Wire Line
+	6600 5650 6200 5650
+Wire Wire Line
+	6200 5650 6200 5700
+Connection ~ 6600 5650
+Wire Wire Line
+	6200 5600 6200 5650
+Wire Wire Line
+	6600 6000 6600 6050
+Wire Wire Line
+	6200 6050 6200 6000
+Wire Wire Line
+	6200 6050 6600 6050
+Connection ~ 6600 6050
+Wire Wire Line
+	6200 6050 6200 6100
+Wire Wire Line
+	7000 6000 7000 6050
+Wire Wire Line
+	7000 6050 6600 6050
 $Comp
 L power:+5V #PWR0119
@@
 L Device:C C11
 U 1 1 60EB05A3
-P 7700 5950
-F 0 "C11" H 7815 5996 50  0000 L CNN
-F 1 "4u7" H 7815 5905 50  0000 L CNN
-F 2 "Capacitor_SMD:C_0603_1608Metric_Pad1.05x0.95mm_HandSolder" H 7738 5800 50  0001 C CNN
-F 3 "~" H 7700 5950 50  0001 C CNN
-	1    7700 5950
-	1    0    0    -1
-$EndComp
-Connection ~ 6450 5750
-Connection ~ 6450 6150
-Wire Wire Line
-	7700 5800 7700 5750
-Wire Wire Line
-	7700 5750 7250 5750
-Connection ~ 7250 5750
-Wire Wire Line
-	7250 6150 7700 6150
-Wire Wire Line
-	7700 6150 7700 6100
-Connection ~ 7250 6150
+P 7450 5850
+F 0 "C11" H 7565 5896 50  0000 L CNN
+F 1 "4u7" H 7565 5805 50  0000 L CNN
+F 2 "Capacitor_SMD:C_0603_1608Metric_Pad1.05x0.95mm_HandSolder" H 7488 5700 50  0001 C CNN
+F 3 "~" H 7450 5850 50  0001 C CNN
+	1    7450 5850
+	1    0    0    -1
+$EndComp
+Connection ~ 6200 5650
+Connection ~ 6200 6050
+Wire Wire Line
+	7450 5700 7450 5650
+Wire Wire Line
+	7450 5650 7000 5650
+Connection ~ 7000 5650
+Wire Wire Line
+	7000 6050 7450 6050
+Wire Wire Line
+	7450 6050 7450 6000
+Connection ~ 7000 6050
 Wire Wire Line
 	5250 1800 5150 1800
@@
 L Device:LED D1
 U 1 1 6123C25B
-P 5800 5650
-F 0 "D1" V 5839 5532 50  0000 R CNN
-F 1 "LED" V 5748 5532 50  0000 R CNN
-F 2 "Diode_SMD:D_0603_1608Metric_Pad1.05x0.95mm_HandSolder" H 5800 5650 50  0001 C CNN
-F 3 "~" H 5800 5650 50  0001 C CNN
-	1    5800 5650
+P 5800 5550
+F 0 "D1" V 5839 5432 50  0000 R CNN
+F 1 "LED" V 5748 5432 50  0000 R CNN
+F 2 "Diode_SMD:D_0603_1608Metric_Pad1.05x0.95mm_HandSolder" H 5800 5550 50  0001 C CNN
+F 3 "~" H 5800 5550 50  0001 C CNN
+	1    5800 5550
 	0    -1   -1   0
 $EndComp
@@
 L Device:R R16
 U 1 1 61245141
-P 5800 6000
-F 0 "R16" H 5870 6046 50  0000 L CNN
-F 1 "300R" H 5870 5955 50  0000 L CNN
-F 2 "Resistor_SMD:R_0603_1608Metric_Pad1.05x0.95mm_HandSolder" V 5730 6000 50  0001 C CNN
-F 3 "~" H 5800 6000 50  0001 C CNN
-	1    5800 6000
+P 5800 5900
+F 0 "R16" H 5870 5946 50  0000 L CNN
+F 1 "300R" H 5870 5855 50  0000 L CNN
+F 2 "Resistor_SMD:R_0603_1608Metric_Pad1.05x0.95mm_HandSolder" V 5730 5900 50  0001 C CNN
+F 3 "~" H 5800 5900 50  0001 C CNN
+	1    5800 5900
 	1    0    0    -1
 $EndComp
@@
 L power:+5V #PWR0120
 U 1 1 6124AFCC
-P 5800 5450
-F 0 "#PWR0120" H 5800 5300 50  0001 C CNN
-F 1 "+5V" H 5815 5623 50  0000 C CNN
-F 2 "" H 5800 5450 50  0001 C CNN
-F 3 "" H 5800 5450 50  0001 C CNN
-	1    5800 5450
+P 5800 5350
+F 0 "#PWR0120" H 5800 5200 50  0001 C CNN
+F 1 "+5V" H 5815 5523 50  0000 C CNN
+F 2 "" H 5800 5350 50  0001 C CNN
+F 3 "" H 5800 5350 50  0001 C CNN
+	1    5800 5350
 	1    0    0    -1
 $EndComp
@@
 L power:Earth #PWR0121
 U 1 1 6124B59D
-P 5800 6200
-F 0 "#PWR0121" H 5800 5950 50  0001 C CNN
-F 1 "Earth" H 5800 6050 50  0001 C CNN
-F 2 "" H 5800 6200 50  0001 C CNN
-F 3 "~" H 5800 6200 50  0001 C CNN
-	1    5800 6200
-	1    0    0    -1
-$EndComp
-Wire Wire Line
-	5800 5850 5800 5800
-Wire Wire Line
-	5800 5450 5800 5500
-Wire Wire Line
-	5800 6200 5800 6150
+P 5800 6100
+F 0 "#PWR0121" H 5800 5850 50  0001 C CNN
+F 1 "Earth" H 5800 5950 50  0001 C CNN
+F 2 "" H 5800 6100 50  0001 C CNN
+F 3 "~" H 5800 6100 50  0001 C CNN
+	1    5800 6100
+	1    0    0    -1
+$EndComp
+Wire Wire Line
+	5800 5750 5800 5700
+Wire Wire Line
+	5800 5350 5800 5400
+Wire Wire Line
+	5800 6100 5800 6050
 Wire Bus Line
 	6200 900  6200 1600
