File: _autosave-luncheonmeat.sch (KiCad schematic (older format))
At the start: 55 parts, among them J1 USB_B_Micro, J2 Conn_02x03_Odd_Even, Q1 Q_PMOS_DGS, Q2 Q_PMOS_DGS, Q3 Q_PMOS_DGS, SW1 SW_Push, SW10 7, SW11 4, SW12 1, SW13 *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

Commit message: late
Parts:
- removed JP? (x2): Jumper_2_Open, symbol Jumper:Jumper_2_Open
Changed lines of the file:
@@
 Text Label 3500 5350 0    50   ~ 0
 DR+
-$Comp
-L Jumper:Jumper_2_Open JP?
-U 1 1 5FE76AA6
-P 3350 3900
-F 0 "JP?" H 3350 4135 50  0000 C CNN
-F 1 "Jumper_2_Open" H 3350 4044 50  0000 C CNN
-F 2 "" H 3350 3900 50  0001 C CNN
-F 3 "~" H 3350 3900 50  0001 C CNN
-	1    3350 3900
-	1    0    0    -1
-$EndComp
-$Comp
-L Jumper:Jumper_2_Open JP?
-U 1 1 5FE77D43
-P 3350 4200
-F 0 "JP?" H 3350 4435 50  0000 C CNN
-F 1 "Jumper_2_Open" H 3350 4344 50  0000 C CNN
-F 2 "" H 3350 4200 50  0001 C CNN
-F 3 "~" H 3350 4200 50  0001 C CNN
-	1    3350 4200
-	1    0    0    -1
-$EndComp
 Wire Bus Line
 	6200 900  6200 1600
@@
 Wire Bus Line
 	8200 1600 8200 6000
-Text GLabel 3150 4200 0    50   Input ~ 0
-TX
-Text GLabel 3550 4200 2    50   Input ~ 0
-TX
-Text GLabel 3550 3900 2    50   Input ~ 0
-RX
-Text GLabel 3150 3900 0    50   Input ~ 0
-RX
 $EndSCHEMATC
