File: luncheonmeat.kicad_pcb (KiCad board)
At the start: 2 copper layers, 37 parts, among them J1 USB_B_Micro, Q1 Q_PMOS_DGS, Q2 Q_PMOS_DGS, Q3 Q_PMOS_DGS, SW1 SW_Push, SW10 9, SW11 6, SW12 3, SW13 #, SW2 7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

Commit message: progress
Parts:
- added C10: 100n, Capacitor_SMD:C_0603_1608Metric_Pad1.05x0.95mm_HandSolder, F.Cu at (120.0, 33.7)
- added C11: 4u7, Capacitor_SMD:C_0603_1608Metric_Pad1.05x0.95mm_HandSolder, F.Cu at (121.9, 31.1)
- added C8: 100n, Capacitor_SMD:C_0603_1608Metric_Pad1.05x0.95mm_HandSolder, F.Cu at (120.7, 47.0)
- added C9: 100n, Capacitor_SMD:C_0603_1608Metric_Pad1.05x0.95mm_HandSolder, F.Cu at (123.8, 33.7)
- added D1: LED, Diode_SMD:D_0603_1608Metric_Pad1.05x0.95mm_HandSolder, F.Cu at (72.9, 42.4)
- added J2: Conn_02x03_Odd_Even, Connector_PinHeader_2.54mm:PinHeader_2x03_P2.54mm_Vertical, F.Cu at (71.1, 32.5)
- added R10: 300R, Resistor_SMD:R_0603_1608Metric_Pad1.05x0.95mm_HandSolder, F.Cu at (97.8, 40.6)
- added R11: 300R, Resistor_SMD:R_0603_1608Metric_Pad1.05x0.95mm_HandSolder, F.Cu at (97.8, 42.5)
- added R12: 300R, Resistor_SMD:R_0603_1608Metric_Pad1.05x0.95mm_HandSolder, F.Cu at (97.8, 44.5)
- added R13: 300R, Resistor_SMD:R_0603_1608Metric_Pad1.05x0.95mm_HandSolder, F.Cu at (97.8, 46.4)
- added R14: 300R, Resistor_SMD:R_0603_1608Metric_Pad1.05x0.95mm_HandSolder, F.Cu at (97.8, 48.3)
- added R15: 300R, Resistor_SMD:R_0603_1608Metric_Pad1.05x0.95mm_HandSolder, F.Cu at (114.3, 46.4)
- added R16: 300R, Resistor_SMD:R_0603_1608Metric_Pad1.05x0.95mm_HandSolder, F.Cu at (72.9, 45.0)
- added R7: 300R, Resistor_SMD:R_0603_1608Metric_Pad1.05x0.95mm_HandSolder, F.Cu at (97.8, 34.9)
- added R8: 300R, Resistor_SMD:R_0603_1608Metric_Pad1.05x0.95mm_HandSolder, F.Cu at (97.8, 36.8)
- added R9: 300R, Resistor_SMD:R_0603_1608Metric_Pad1.05x0.95mm_HandSolder, F.Cu at (97.8, 38.7)
- J1: footprint Connector_USB:USB_Micro-B_Molex-105017-0001 -> Connector_USB:USB_Micro-B_Wuerth_629105150521_CircularHoles
- R1: value R -> 100k
- R2, R3, R4: footprint Resistor_SMD:R_0201_0603Metric -> Resistor_SMD:R_0603_1608Metric_Pad1.05x0.95mm_HandSolder
- SW10: value 9 -> 7
- SW11: value 6 -> 4
- SW12: value 3 -> 1
- SW13: value # -> *
- SW2: value 7 -> 9
- SW3: value 4 -> 6
- SW4: value 1 -> 3
- SW5: value * -> #
- Y1: value Crystal -> 16MHz; footprint Crystal:Crystal_HC49-U_Vertical -> Crystal:Crystal_HC49-4H_Vertical
- moved R2 78.1 mm to (68.6, 61.0), turned to 270 degrees
- moved Q1 76.0 mm to (71.1, 61.0), turned to 90 degrees
- moved SW13 69.0 mm to (82.1, 172.2)
- moved SW10 66.2 mm to (82.1, 112.2)
- moved SW12 65.9 mm to (82.1, 152.2)
- moved SW11 65.0 mm to (82.1, 132.2)
- moved Q3 57.7 mm to (94.0, 61.0), turned to 90 degrees
- moved R6 45.0 mm to (106.0, 35.6), turned to 270 degrees
- moved R5 43.7 mm to (108.6, 35.6), turned to 270 degrees
- moved C5 43.7 mm to (105.4, 33.0)
- moved SW9 42.0 mm to (102.1, 172.2)
- moved U2 41.8 mm to (66.0, 63.5)
- moved C6 41.2 mm to (109.2, 33.0)
- moved R3 41.0 mm to (114.3, 61.0), turned to 270 degrees
- moved U4 40.6 mm to (91.4, 63.5)
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Connections:
- U1 pad 1: /SEG_D -> Net-(R14-Pad2)
- U1 pad 10: /SEG_G -> /SEG_SEL_2
- U1 pad 11: /SEG_RDP -> Net-(U1-Pad11)
- U1 pad 12: /ROW_0 -> /COL_0
- U1 pad 13: /ROW_1 -> /COL_1
- U1 pad 14: /ROW_2 -> /COL_2
- U1 pad 15: /ROW_3 -> MOSI
- U1 pad 16: Net-(U1-Pad16) -> MISO
- U1 pad 17: Net-(U1-Pad17) -> SCK
- U1 pad 18: Net-(U1-Pad18) -> +5V
- U1 pad 19: /COL_2 -> /ROW_2
- U1 pad 2: /SEG_E -> /SEG_SEL_0
- U1 pad 20: Net-(U1-Pad20) -> +5V
- U1 pad 21: Net-(U1-Pad21) -> Earth
- U1 pad 22: Net-(U1-Pad22) -> /ROW_3
- U1 pad 23: /SEG_SEL_0 -> Net-(R7-Pad2)
- U1 pad 24: /SEG_SEL_1 -> Net-(R8-Pad2)
- U1 pad 25: /SEG_SEL_2 -> Net-(R9-Pad2)
- U1 pad 29: Net-(C1-Pad2) -> RESET
- U1 pad 3: /COL_0 -> /ROW_0
- U1 pad 30: /SEG_A -> RX
- U1 pad 31: /SEG_B -> TX
- U1 pad 32: /SEG_C -> Net-(R13-Pad2)
- U1 pad 4: Net-(U1-Pad4) -> +5V
- U1 pad 5: Net-(U1-Pad21) -> Earth
- U1 pad 6: /COL_1 -> /ROW_1
- U1 pad 9: /SEG_F -> /SEG_SEL_1
- U5 pad 1: Net-(U5-Pad1) -> TX
- U5 pad 4: Net-(U5-Pad4) -> RX

Commit message: progress
Parts:
- moved D1 54.6 mm to (127.0, 50.0)
- moved R16 54.2 mm to (127.0, 48.0), turned to 180 degrees
- moved R14 41.8 mm to (136.0, 65.3), turned to 90 degrees
- moved J2 41.5 mm to (109.1, 49.3)
- moved R13 40.9 mm to (134.1, 65.3), turned to 90 degrees
- moved R12 40.2 mm to (132.2, 65.3), turned to 90 degrees
- moved R11 39.7 mm to (130.3, 65.3), turned to 90 degrees
- moved R10 39.3 mm to (128.4, 65.3), turned to 90 degrees
- moved U2 39.3 mm to (95.0, 90.0)
- moved R7 39.2 mm to (122.6, 65.3), turned to 90 degrees
- moved R9 39.1 mm to (126.5, 65.3), turned to 90 degrees
- moved R8 39.1 mm to (124.5, 65.3), turned to 90 degrees
- moved U4 39.0 mm to (120.0, 90.0)
- moved U3 38.7 mm to (145.0, 90.0)
- moved U1 27.4 mm to (141.6, 57.7)
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
Commit message: progress
Parts:
- SW1: footprint Button_Switch_THT:SW_PUSH_6mm -> Connector_PinHeader_2.54mm:PinHeader_1x02_P2.54mm_Vertical
- moved C11 49.0 mm to (95.2, 60.4), turned to 180 degrees
- moved C9 47.5 mm to (97.7, 58.5), turned to 90 degrees
- moved C10 44.6 mm to (97.7, 62.3), turned to 270 degrees
- moved U1 37.7 mm to (104.1, 61.6), turned to 180 degrees
- moved C3 37.0 mm to (110.4, 56.6), turned to 90 degrees
- moved C2 32.6 mm to (110.4, 60.4), turned to 90 degrees
- moved R12 30.2 mm to (102.3, 69.8)
- moved R13 30.2 mm to (104.2, 69.8)
- moved R14 30.2 mm to (106.1, 69.8)
- moved R7 30.2 mm to (92.8, 69.8)
- moved R8 30.2 mm to (94.7, 69.8)
- moved R9 30.2 mm to (96.6, 69.8)
- moved R10 30.2 mm to (98.5, 69.8)
- moved R11 30.2 mm to (100.4, 69.8)
- moved Y1 28.8 mm to (114.2, 61.0), turned to 90 degrees
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
Commit message: progress
Parts:
- moved R2 2.90 mm to (87.6, 69.8)
- moved Q1 2.89 mm to (90.2, 69.8)
- moved Q3 0.66 mm to (110.5, 69.8)
- moved R4 0.66 mm to (108.0, 69.8)
- moved R3 0.16 mm to (133.3, 69.8)
- moved R14 0.13 mm to (106.0, 69.8)
- moved Q2 0.11 mm to (136.0, 69.8)
- moved R10 0.09 mm to (98.4, 69.8)
- moved R11 0.09 mm to (100.3, 69.8)
- moved R8 0.09 mm to (94.6, 69.8)
- moved R9 0.09 mm to (96.5, 69.8)
- moved R12 0.08 mm to (102.2, 69.8)
- moved R13 0.08 mm to (104.1, 69.8)
Changed lines of the file:
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@@
   )
   (module Resistor_SMD:R_0603_1608Metric_Pad1.05x0.95mm_HandSolder (layer F.Cu)
-    (at 106.13 69.75 90)
+    (at 106.045 69.85 90)
     (descr "Resistor SMD 0603 (1608 Metric), square (rectangular) end terminal, IPC_7351 nominal with elongated pad for handsoldering. (Body size source: http://www.tortai-tech.com/upload/download/2011102023233369053.pdf), generated with kicad-footprint-generator")
     (tags "resistor handsolder")
@@
   )
   (module Resistor_SMD:R_0603_1608Metric_Pad1.05x0.95mm_HandSolder (layer F.Cu)
-    (at 104.225 69.75 90)
+    (at 104.14 69.75 90)
     (descr "Resistor SMD 0603 (1608 Metric), square (rectangular) end terminal, IPC_7351 nominal with elongated pad for handsoldering. (Body size source: http://www.tortai-tech.com/upload/download/2011102023233369053.pdf), generated with kicad-footprint-generator")
     (tags "resistor handsolder")
@@
   )
   (module Resistor_SMD:R_0603_1608Metric_Pad1.05x0.95mm_HandSolder (layer F.Cu)
-    (at 102.32 69.75 90)
+    (at 102.235 69.75 90)
     (descr "Resistor SMD 0603 (1608 Metric), square (rectangular) end terminal, IPC_7351 nominal with elongated pad for handsoldering. (Body size source: http://www.tortai-tech.com/upload/download/2011102023233369053.pdf), generated with kicad-footprint-generator")
     (tags "resistor handsolder")
@@
   )
   (module Resistor_SMD:R_0603_1608Metric_Pad1.05x0.95mm_HandSolder (layer F.Cu)
-    (at 100.415 69.75 90)
+    (at 100.33 69.75 90)
     (descr "Resistor SMD 0603 (1608 Metric), square (rectangular) end terminal, IPC_7351 nominal with elongated pad for handsoldering. (Body size source: http://www.tortai-tech.com/upload/download/2011102023233369053.pdf), generated with kicad-footprint-generator")
     (tags "resistor handsolder")
@@
   )
   (module Resistor_SMD:R_0603_1608Metric_Pad1.05x0.95mm_HandSolder (layer F.Cu)
-    (at 98.51 69.75 90)
+    (at 98.425 69.75 90)
     (descr "Resistor SMD 0603 (1608 Metric), square (rectangular) end terminal, IPC_7351 nominal with elongated pad for handsoldering. (Body size source: http://www.tortai-tech.com/upload/download/2011102023233369053.pdf), generated with kicad-footprint-generator")
     (tags "resistor handsolder")
@@
   )
   (module Resistor_SMD:R_0603_1608Metric_Pad1.05x0.95mm_HandSolder (layer F.Cu)
-    (at 96.605 69.75 90)
+    (at 96.52 69.75 90)
     (descr "Resistor SMD 0603 (1608 Metric), square (rectangular) end terminal, IPC_7351 nominal with elongated pad for handsoldering. (Body size source: http://www.tortai-tech.com/upload/download/2011102023233369053.pdf), generated with kicad-footprint-generator")
     (tags "resistor handsolder")
@@
   )
   (module Resistor_SMD:R_0603_1608Metric_Pad1.05x0.95mm_HandSolder (layer F.Cu)
-    (at 94.7 69.75 90)
+    (at 94.615 69.75 90)
     (descr "Resistor SMD 0603 (1608 Metric), square (rectangular) end terminal, IPC_7351 nominal with elongated pad for handsoldering. (Body size source: http://www.tortai-tech.com/upload/download/2011102023233369053.pdf), generated with kicad-footprint-generator")
     (tags "resistor handsolder")
@@
   )
   (module Resistor_SMD:R_0603_1608Metric_Pad1.05x0.95mm_HandSolder (layer F.Cu)
-    (at 108.6 69.96 270)
+    (at 107.95 69.85 270)
     (descr "Resistor SMD 0603 (1608 Metric), square (rectangular) end terminal, IPC_7351 nominal with elongated pad for handsoldering. (Body size source: http://www.tortai-tech.com/upload/download/2011102023233369053.pdf), generated with kicad-footprint-generator")
     (tags "resistor handsolder")
@@
   )
   (module Resistor_SMD:R_0603_1608Metric_Pad1.05x0.95mm_HandSolder (layer F.Cu)
-    (at 133.46 69.96 270)
+    (at 133.35 69.85 270)
     (descr "Resistor SMD 0603 (1608 Metric), square (rectangular) end terminal, IPC_7351 nominal with elongated pad for handsoldering. (Body size source: http://www.tortai-tech.com/upload/download/2011102023233369053.pdf), generated with kicad-footprint-generator")
     (tags "resistor handsolder")
@@
   )
   (module Resistor_SMD:R_0603_1608Metric_Pad1.05x0.95mm_HandSolder (layer F.Cu)
-    (at 84.74 69.96 270)
+    (at 87.63 69.75 270)
     (descr "Resistor SMD 0603 (1608 Metric), square (rectangular) end terminal, IPC_7351 nominal with elongated pad for handsoldering. (Body size source: http://www.tortai-tech.com/upload/download/2011102023233369053.pdf), generated with kicad-footprint-generator")
     (tags "resistor handsolder")
@@
   )
   (module Package_TO_SOT_SMD:SOT-23 (layer F.Cu)
-    (at 111.14 69.96 90)
+    (at 110.49 69.85 90)
     (descr "SOT-23, Standard")
     (tags SOT-23)
@@
   )
   (module Package_TO_SOT_SMD:SOT-23 (layer F.Cu)
-    (at 136 69.96 90)
+    (at 136 69.85 90)
     (descr "SOT-23, Standard")
     (tags SOT-23)
@@
   )
   (module Package_TO_SOT_SMD:SOT-23 (layer F.Cu)
-    (at 87.28 69.96 90)
+    (at 90.17 69.85 90)
     (descr "SOT-23, Standard")
     (tags SOT-23)

Commit message: late
Parts:
- moved C7 7.65 mm to (128.8, 66.6)
- moved C1 6.85 mm to (76.9, 63.8), turned to 0 degrees
- moved R1 5.86 mm to (76.9, 65.3), turned to 0 degrees
- moved SW1 4.81 mm to (80.5, 62.1)
- moved R15 4.81 mm to (80.5, 65.3)
- moved J2 4.81 mm to (84.2, 57.0)
- moved C10 4.75 mm to (93.5, 60.1), turned to 180 degrees
- moved C9 4.44 mm to (93.5, 57.1), turned to 180 degrees
- moved U1 3.41 mm to (101.5, 59.4)
- moved C11 2.45 mm to (93.5, 58.6)
- moved C8 2.33 mm to (110.0, 61.9)
- moved C2 2.11 mm to (110.0, 58.3)
- moved Y1 2.05 mm to (113.8, 59.0)
- moved C3 1.71 mm to (110.0, 54.9)
- moved C4 0.50 mm to (129.2, 59.5)
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Connections:
- net Net-(C5-Pad2) renamed /D+
- net Net-(C6-Pad1) renamed /D-
- net Net-(R5-Pad2) renamed /DR-
- net Net-(R6-Pad2) renamed /DR+
- R3 pad 1: /SEG_SEL_0 -> /SEG_SEL_1
- R4 pad 1: /SEG_SEL_0 -> /SEG_SEL_2
Routing:
- net /COL_0: track 0.00 -> 210.4 mm, vias 0 -> 1
- net /COL_1: track 0.00 -> 191.4 mm, vias 0 -> 1
- net /ROW_3: track 0.00 -> 182.4 mm, vias 0 -> 1
- net /COL_2: track 0.00 -> 172.4 mm, vias 0 -> 1
- net /ROW_2: track 0.00 -> 164.1 mm, vias 0 -> 2
- net /ROW_1: track 0.00 -> 149.2 mm
- net /ROW_0: track 0.00 -> 124.9 mm
- net /SEG_D: track 0.00 -> 107.3 mm
- net /SEG_C: track 0.00 -> 107.3 mm
- net /SEG_E: track 0.00 -> 100.5 mm
- net /SEG_RDP: track 0.00 -> 90.9 mm
- net +5V: track 0.00 -> 68.6 mm, vias 0 -> 1
- net /SEG_SEL_1: track 0.00 -> 43.1 mm
- net Net-(Q1-Pad2): track 0.00 -> 36.6 mm, vias 0 -> 1
- net /SEG_A: track 0.00 -> 35.3 mm, vias 0 -> 2
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