File: hardware/luncheonmeat.kicad_pcb (KiCad board)
At the start: 2 copper layers, 53 parts, among them J1 USB_B_Micro, J2 Conn_02x03_Odd_Even, Q1 Q_PMOS_DGS, Q2 Q_PMOS_DGS, Q3 Q_PMOS_DGS, SW1 SW_Push, SW10 7, SW11 4, SW12 1, SW13 *, SW2 9, SW3 6, SW4 3, SW5 #, SW6 8, SW7 5, SW8 2, SW9 0, U1 ATmega328PB-AU, U2 lsd100bag-101-20, U3 lsd100bag-101-20, U4 lsd100bag-101-20, U5 FT230XS, Y1 16MHz

Commit message: Fix schematic, new board layout
Parts:
- added C12: 22pF, Capacitor_SMD:C_0603_1608Metric_Pad1.08x0.95mm_HandSolder, F.Cu at (90.5, 92.5)
- added C13: 22pF, Capacitor_SMD:C_0603_1608Metric_Pad1.08x0.95mm_HandSolder, F.Cu at (92.9, 82.6)
- added D2: R, LED_SMD:LED_0805_2012Metric_Castellated, F.Cu at (152.2, 66.8)
- added D3: Y, LED_SMD:LED_0805_2012Metric_Castellated, F.Cu at (152.2, 69.8)
- added D4: D_Small, Diode_SMD:D_0805_2012Metric, F.Cu at (114.5, 68.5)
- added H1: MH, MountingHole:MountingHole_3.2mm_M3_DIN965, F.Cu at (86.0, 67.5)
- added H2: MH, MountingHole:MountingHole_3.2mm_M3_DIN965, F.Cu at (86.0, 111.0)
- added H3: MH, MountingHole:MountingHole_3.2mm_M3_DIN965, F.Cu at (86.0, 190.0)
- added H4: MH, MountingHole:MountingHole_3.2mm_M3_DIN965, F.Cu at (161.0, 67.5)
- added H5: MH, MountingHole:MountingHole_3.2mm_M3_DIN965, F.Cu at (161.0, 111.5)
- added H6: MH, MountingHole:MountingHole_3.2mm_M3_DIN965, F.Cu at (161.0, 190.0)
- added R17: 0R, Resistor_SMD:R_0805_2012Metric_Pad1.20x1.40mm_HandSolder, F.Cu at (129.5, 89.5)
- added R18: 0R, Resistor_SMD:R_0805_2012Metric_Pad1.20x1.40mm_HandSolder, F.Cu at (129.5, 92.0)
- added R19: 1k, Resistor_SMD:R_0805_2012Metric_Pad1.20x1.40mm_HandSolder, F.Cu at (153.0, 79.5)
- added R20: 1k, Resistor_SMD:R_0805_2012Metric_Pad1.20x1.40mm_HandSolder, F.Cu at (127.0, 79.0)
- added R21: 1k, Resistor_SMD:R_0805_2012Metric_Pad1.20x1.40mm_HandSolder, F.Cu at (101.0, 78.5)
- C1: value 100n -> 10nF; footprint Capacitor_SMD:C_0603_1608Metric_Pad1.05x0.95mm_HandSolder -> Capacitor_SMD:C_0805_2012Metric_Pad1.18x1.45mm_HandSolder
- C10, C7, C8, C9: value 100n -> 100nF; footprint Capacitor_SMD:C_0603_1608Metric_Pad1.05x0.95mm_HandSolder -> Capacitor_SMD:C_0805_2012Metric_Pad1.18x1.45mm_HandSolder
- C2: value 22p -> 10nF; footprint Capacitor_SMD:C_0603_1608Metric_Pad1.05x0.95mm_HandSolder -> Capacitor_SMD:C_0805_2012Metric_Pad1.18x1.45mm_HandSolder
- C3: value 22p -> 47p; footprint Capacitor_SMD:C_0603_1608Metric_Pad1.05x0.95mm_HandSolder -> Capacitor_SMD:C_0805_2012Metric_Pad1.18x1.45mm_HandSolder
- C4: value 10n -> 47p; footprint Capacitor_SMD:C_0603_1608Metric_Pad1.05x0.95mm_HandSolder -> Capacitor_SMD:C_0805_2012Metric_Pad1.18x1.45mm_HandSolder
- C5, C6: value 47p -> 100nF; footprint Capacitor_SMD:C_0603_1608Metric_Pad1.05x0.95mm_HandSolder -> Capacitor_SMD:C_0805_2012Metric_Pad1.18x1.45mm_HandSolder
- D1: value LED -> G; footprint Diode_SMD:D_0603_1608Metric_Pad1.05x0.95mm_HandSolder -> LED_SMD:LED_0805_2012Metric_Castellated
- J2: value Conn_02x03_Odd_Even -> AVR-ISP-6; footprint Connector_PinHeader_2.54mm:PinHeader_2x03_P2.54mm_Vertical -> Connector_IDC:IDC-Header_2x03_P2.54mm_Vertical
- R1: value 100k -> 1M; footprint Resistor_SMD:R_0603_1608Metric_Pad1.05x0.95mm_HandSolder -> Resistor_SMD:R_0805_2012Metric_Pad1.20x1.40mm_HandSolder
- R10, R11, R12, R13, R14, R15, R16, R5, R6, R7, R9: footprint Resistor_SMD:R_0603_1608Metric_Pad1.05x0.95mm_HandSolder -> Resistor_SMD:R_0805_2012Metric_Pad1.20x1.40mm_HandSolder
- R2: value 1k -> 300R; footprint Resistor_SMD:R_0603_1608Metric_Pad1.05x0.95mm_HandSolder -> Resistor_SMD:R_0805_2012Metric_Pad1.20x1.40mm_HandSolder
- R3, R4: value 1k -> 1.5k; footprint Resistor_SMD:R_0603_1608Metric_Pad1.05x0.95mm_HandSolder -> Resistor_SMD:R_0805_2012Metric_Pad1.20x1.40mm_HandSolder
- R8: value 300R -> 10k; footprint Resistor_SMD:R_0603_1608Metric_Pad1.05x0.95mm_HandSolder -> Resistor_SMD:R_0805_2012Metric_Pad1.20x1.40mm_HandSolder
- SW1: value SW_Push -> 7; footprint Connector_PinHeader_2.54mm:PinHeader_1x02_P2.54mm_Vertical -> Button_Switch_THT:SW_PUSH_6mm
- SW10: value 7 -> 6
- SW11: value 4 -> 3
- SW12: value 1 -> #
- SW13: value * -> SW_Push; footprint Button_Switch_THT:SW_PUSH_6mm -> Button_Switch_SMD:SW_Push_1P1T_NO_CK_KSC7xxJ
- SW2: value 9 -> 4
- SW3: value 6 -> 1
- SW4: value 3 -> *
- SW5: value # -> 8
- SW6: value 8 -> 5
- SW7: value 5 -> 2
- SW8: value 2 -> 0
- SW9: value 0 -> 9
- U2: value lsd100bag-101-20 -> FT230XS; footprint lsd100bag-101-20:lsd100bag-101-20 -> Package_SO:SSOP-16_3.9x4.9mm_P0.635mm
- U5: value FT230XS -> lsd100bag-101-20; footprint Package_SO:SSOP-16_3.9x4.9mm_P0.635mm -> lsd100bag-101-20:lsd100bag-101-20
- Y1: value 16MHz -> 8MHz; footprint Crystal:Crystal_HC49-4H_Vertical -> Crystal:Crystal_SMD_0603-4Pin_6.0x3.5mm_HandSoldering
- moved SW13 109.4 mm to (101.5, 68.5), turned to 180 degrees
- moved J2 64.0 mm to (87.0, 121.0)
- moved SW9 62.3 mm to (140.0, 120.0)
- moved SW1 61.1 mm to (100.0, 120.0), turned to 0 degrees
- moved SW5 60.1 mm to (120.0, 120.0)
- moved Q1 60.1 mm to (149.5, 79.5), turned to 180 degrees
- moved C10 55.2 mm to (143.5, 83.5), turned to 0 degrees
- moved C1 51.0 mm to (127.5, 70.0)
- moved R1 50.6 mm to (127.5, 67.0), turned to 180 degrees
- moved SW11 48.6 mm to (140.0, 160.0)
- moved SW12 48.6 mm to (140.0, 180.0)
- moved SW10 48.6 mm to (140.0, 140.0)
- moved C9 46.8 mm to (129.5, 87.0)
- moved SW2 43.0 mm to (100.0, 140.0)
- moved SW3 43.0 mm to (100.0, 160.0)
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Connections:
- C1 pad 1: Earth -> GND
- C10 pad 2: Earth -> GND
- C11 pad 2: Earth -> GND
- C2 pad 1: Earth -> GND
- C3 pad 1: Net-(C3-Pad1) -> GND
- C3 pad 2: Earth -> /D+
- C4 pad 1: Earth -> /D-
- C4 pad 2: Net-(C4-Pad2) -> GND
- C5 pad 1: Earth -> GND
- C5 pad 2: /D+ -> +5VD
- C6 pad 1: /D- -> GND
- C6 pad 2: Earth -> +5V
- C7 pad 1: Earth -> GND
- C8 pad 1: +5V -> GND
- C8 pad 2: Earth -> +5V
- C9 pad 2: Earth -> GND
- D1 pad 1: Net-(D1-Pad1) -> GND
- D1 pad 2: +5V -> Net-(D1-Pad2)
- J1 pad 1: Net-(C4-Pad2) -> Net-(C2-Pad2)
- J1 pad 5: Earth -> GND
- J1 pad 6: Net-(J1-Pad6) -> Net-(C1-Pad2)
- J2 pad 6: Earth -> GND
- L1 pad 1: Net-(C4-Pad2) -> Net-(C2-Pad2)
- R1 pad 1: +5V -> Net-(C1-Pad2)
- R1 pad 2: Net-(C1-Pad2) -> GND
- R11 pad 1: /SEG_E -> /SEG_C
- R12 pad 1: /SEG_F -> /SEG_RDP
- R13 pad 1: /SEG_G -> /SEG_F
- R14 pad 1: /SEG_RDP -> /SEG_G
- R15 pad 1: Net-(C1-Pad2) -> /SEG_B
- R15 pad 2: RESET -> Net-(R15-Pad2)
- R16 pad 1: Net-(D1-Pad1) -> /SEG_A
- R16 pad 2: Earth -> Net-(R16-Pad2)
- R2 pad 1: /SEG_SEL_0 -> Net-(D1-Pad2)
- R2 pad 2: Net-(Q1-Pad1) -> P_LED
- R3 pad 1: /SEG_SEL_1 -> Net-(D2-Pad2)
- R3 pad 2: Net-(Q2-Pad1) -> +5VD
- R4 pad 1: /SEG_SEL_2 -> Net-(D3-Pad2)
- R4 pad 2: Net-(Q3-Pad1) -> +5VD
- R7 pad 1: /SEG_A -> Net-(C7-Pad2)
- R7 pad 2: Net-(R7-Pad2) -> RESET
- R8 pad 1: /SEG_B -> Net-(C7-Pad2)
- R8 pad 2: Net-(R8-Pad2) -> +5V
- R9 pad 1: /SEG_C -> /SEG_E
- SW1 pad 1: Net-(C1-Pad2) -> /ROW_0
- SW1 pad 2: Earth -> /COL_2
- SW10 pad 1: /ROW_0 -> /ROW_1
- SW10 pad 2: /COL_2 -> /COL_0
- SW11 pad 1: /ROW_1 -> /ROW_2
- SW11 pad 2: /COL_2 -> /COL_0
- SW12 pad 1: /ROW_2 -> /ROW_3
- SW12 pad 2: /COL_2 -> /COL_0
- SW13 pad 1: /ROW_3 -> Net-(C7-Pad2)
- SW13 pad 2: /COL_2 -> GND
- SW2 pad 1: /ROW_0 -> /ROW_1
- SW2 pad 2: /COL_0 -> /COL_2
- SW3 pad 1: /ROW_1 -> /ROW_2
- SW3 pad 2: /COL_0 -> /COL_2
- SW4 pad 1: /ROW_2 -> /ROW_3
- SW4 pad 2: /COL_0 -> /COL_2
- SW5 pad 1: /ROW_3 -> /ROW_0
- SW5 pad 2: /COL_0 -> /COL_1
- SW6 pad 1: /ROW_0 -> /ROW_1
- SW7 pad 1: /ROW_1 -> /ROW_2
- SW8 pad 1: /ROW_2 -> /ROW_3
- SW9 pad 1: /ROW_3 -> /ROW_0
- SW9 pad 2: /COL_1 -> /COL_0
- U1 pad 1: Net-(R14-Pad2) -> Net-(R16-Pad2)
- U1 pad 11: Net-(U1-Pad11) -> P_LED
- U1 pad 21: Earth -> GND
- U1 pad 23: Net-(R7-Pad2) -> Net-(R9-Pad2)
- U1 pad 24: Net-(R8-Pad2) -> Net-(R10-Pad2)
- U1 pad 25: Net-(R9-Pad2) -> Net-(R11-Pad2)
- U1 pad 26: Net-(R10-Pad2) -> Net-(R12-Pad2)
- U1 pad 27: Net-(R11-Pad2) -> Net-(R13-Pad2)
- U1 pad 28: Net-(R12-Pad2) -> Net-(R14-Pad2)
- U1 pad 30: RX -> RXD
- U1 pad 31: TX -> TXD
- U1 pad 32: Net-(R13-Pad2) -> Net-(R15-Pad2)
- U1 pad 5: Earth -> GND
- U1 pad 7: Net-(C2-Pad2) -> Net-(C13-Pad1)
- U1 pad 8: Net-(C3-Pad1) -> Net-(C12-Pad2)
- U2 pad 1: /SEG_E -> TX_F
- U2 pad 10: /SEG_G -> +5VD
- U2 pad 2: /SEG_D -> Net-(U2-Pad2)
- U2 pad 3: Net-(Q1-Pad2) -> +5VD
- U2 pad 4: /SEG_C -> RX_F
- U2 pad 5: /SEG_RDP -> GND
- U2 pad 6: /SEG_B -> Net-(U2-Pad6)
- U2 pad 7: /SEG_A -> Net-(U2-Pad7)
- U2 pad 8: Net-(Q1-Pad2) -> /DR+
- U2 pad 9: /SEG_F -> /DR-
- U3 pad 3: Net-(Q2-Pad2) -> Net-(Q1-Pad2)
- U3 pad 8: Net-(Q2-Pad2) -> Net-(Q1-Pad2)
- U4 pad 3: Net-(Q3-Pad2) -> Net-(Q2-Pad2)
- U4 pad 8: Net-(Q3-Pad2) -> Net-(Q2-Pad2)
- U5 pad 1: TX -> /SEG_E
- U5 pad 10: Net-(C7-Pad2) -> /SEG_G
- U5 pad 2: Net-(U5-Pad2) -> /SEG_D
- U5 pad 3: Net-(C7-Pad2) -> Net-(Q3-Pad2)
- U5 pad 4: RX -> /SEG_C
- U5 pad 5: Earth -> /SEG_RDP
- U5 pad 6: Net-(U5-Pad6) -> /SEG_B
- U5 pad 7: Net-(U5-Pad7) -> /SEG_A
- U5 pad 8: /DR+ -> Net-(Q3-Pad2)
- U5 pad 9: /DR- -> /SEG_F
- Y1 pad 1: Net-(C2-Pad2) -> Net-(C12-Pad2)
- Y1 pad 2: Net-(C3-Pad1) -> GND
Routing:
- net /COL_0: track 210.4 -> 0.00 mm, vias 1 -> 0
- net /COL_1: track 191.4 -> 0.00 mm, vias 1 -> 0
- net /ROW_3: track 182.4 -> 0.00 mm, vias 1 -> 0
- net /COL_2: track 172.4 -> 0.00 mm, vias 1 -> 0
- net /ROW_2: track 164.1 -> 0.00 mm, vias 2 -> 0
- net /ROW_1: track 149.2 -> 0.00 mm
- net /ROW_0: track 124.9 -> 0.00 mm
- net +5V: track 68.6 -> 0.00 mm, vias 1 -> 0
- net /SEG_D: track 107.3 -> 57.7 mm
- net /SEG_C: track 107.3 -> 57.7 mm
- net /SEG_B: track 7.19 -> 56.8 mm, vias 1 -> 0
- net /SEG_SEL_1: track 43.1 -> 0.00 mm
- net /SEG_F: track 14.4 -> 57.3 mm, vias 1 -> 0
- net /SEG_E: track 100.5 -> 57.6 mm
- net /SEG_G: track 19.2 -> 56.4 mm, vias 1 -> 0
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Other:
- board outline added: 81 x 128.5 mm
- net class Default: clearance 0.2 -> 0.3; trace_width 0.25 -> 0.3; via_dia 0.8 -> 0.6
- net class Power added: clearance 0.5, trace_width 0.8, via_dia 0.9, via_drill 0.6
- net class Signals added: clearance 0.3, trace_width 0.3, via_dia 0.6, via_drill 0.4
- rule trace_clearance: 0.2 -> 0.3

Commit message: v0.2.0, PCB board finished
Parts:
- added G***: LOGO, logo:logo, B.Cu at (142.7, 172.0)
- added REF**: KiCad-Logo2_5mm_SilkScreen, Symbol:KiCad-Logo2_5mm_SilkScreen, B.Cu at (102.0, 189.2)
- added REF**: WEEE-Logo_4.2x6mm_SilkScreen, Symbol:WEEE-Logo_4.2x6mm_SilkScreen, B.Cu at (90.6, 189.2)
- moved C12 7.42 mm to (89.9, 85.1), turned to 45 degrees
- moved R21 6.50 mm to (94.5, 78.5), turned to 90 degrees
- moved C8 4.72 mm to (102.5, 80.0), turned to 0 degrees
- moved C3 4.56 mm to (134.0, 77.0), turned to 0 degrees
- moved C4 4.03 mm to (138.5, 77.0), turned to 0 degrees
- moved R6 2.50 mm to (135.0, 80.5)
- moved R5 2.00 mm to (137.5, 80.5)
- moved Y1 0.72 mm to (94.0, 86.8)
- moved Q3 0.50 mm to (98.0, 78.5)
- moved C13 0.39 mm to (92.5, 82.5)
- moved R8 0.25 mm to (111.5, 68.5), turned to 270 degrees
- turned D4 to 90 degrees
Connections:
- net Net-(C2-Pad2) renamed /USB+5V
- R15 pad 2: Net-(R15-Pad2) -> /SEG_B_
- R16 pad 2: Net-(R16-Pad2) -> /SEG_A_
- R5 pad 2: /DR- -> /DR+
- R6 pad 2: /DR+ -> /DR-
- SW10 pad 2: /COL_0 -> MISO
- SW11 pad 2: /COL_0 -> MISO
- SW12 pad 2: /COL_0 -> MISO
- SW5 pad 2: /COL_1 -> MOSI
- SW6 pad 2: /COL_1 -> MOSI
- SW7 pad 2: /COL_1 -> MOSI
- SW8 pad 2: /COL_1 -> MOSI
- SW9 pad 2: /COL_0 -> MISO
- U1 pad 1: Net-(R16-Pad2) -> Net-(R13-Pad2)
- U1 pad 10: /SEG_SEL_2 -> /ROW_3
- U1 pad 11: P_LED -> /ROW_2
- U1 pad 12: /COL_0 -> /ROW_1
- U1 pad 13: /COL_1 -> /ROW_0
- U1 pad 19: /ROW_2 -> Net-(U1-Pad19)
- U1 pad 2: /SEG_SEL_0 -> Net-(R14-Pad2)
- U1 pad 22: /ROW_3 -> Net-(U1-Pad22)
- U1 pad 23: Net-(R9-Pad2) -> P_LED
- U1 pad 24: Net-(R10-Pad2) -> Net-(R9-Pad2)
- U1 pad 25: Net-(R11-Pad2) -> Net-(R10-Pad2)
- U1 pad 26: Net-(R12-Pad2) -> Net-(R11-Pad2)
- U1 pad 27: Net-(R13-Pad2) -> Net-(R12-Pad2)
- U1 pad 28: Net-(R14-Pad2) -> /SEG_SEL_0
- U1 pad 3: /ROW_0 -> /SEG_B_
- U1 pad 32: Net-(R15-Pad2) -> /SEG_SEL_1
- U1 pad 6: /ROW_1 -> /SEG_A_
- U1 pad 9: /SEG_SEL_1 -> /SEG_SEL_2
Routing:
- net MISO: track 0.00 -> 230.9 mm
- net MOSI: track 0.00 -> 184.3 mm
- net +5V: track 0.00 -> 167.6 mm, vias 0 -> 9
- net /ROW_3: track 0.00 -> 143.9 mm
- net /COL_2: track 0.00 -> 137.8 mm
- net /ROW_2: track 0.00 -> 123.1 mm
- net /ROW_1: track 0.00 -> 105.1 mm
- net /ROW_0: track 0.00 -> 82.7 mm
- net RESET: track 0.00 -> 81.0 mm, vias 0 -> 3
- net GND: track 0.00 -> 63.1 mm, vias 0 -> 70
- net +5VD: track 0.00 -> 62.5 mm, vias 0 -> 4
- net /SEG_SEL_0: track 0.00 -> 61.3 mm
- net TX_F: track 0.00 -> 51.7 mm, vias 0 -> 2
- net P_LED: track 0.00 -> 51.4 mm, vias 0 -> 2
- net RX_F: track 0.00 -> 48.3 mm, vias 0 -> 2
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- added copper zone on B.Cu, net GND
- added copper zone on F.Cu, net GND
Other:
- net class Power: clearance 0.5 -> 0.3
- net class sSignals added: clearance 0.1, trace_width 0.3, via_dia 0.6, via_drill 0.4
- board text added: "Luncheonmeat"
- board text added: "v0.2.0, Dec 2020"

Commit message: v0.2.1 PCB Updated
Connections:
- net +5VD renamed +3V3
- R5 pad 2: /DR+ -> /DR-
- R6 pad 2: /DR- -> /DR+
Routing:
- net /DR+: track 4.42 -> 6.04 mm
- net /DR-: track 4.21 -> 5.54 mm, vias 0 -> 2

Commit message: v0.2.2 PCB Updated
Parts:
- moved REF** 39.2 mm to (141.2, 189.2), turned to 180 degrees
- moved REF** 39.1 mm to (129.8, 189.2)
- moved R20 5.70 mm to (123.5, 83.5)
- moved R19 5.51 mm to (149.5, 83.8)
- moved Q1 1.03 mm to (150.5, 79.2), turned to 90 degrees
- moved Q2 1.03 mm to (124.5, 78.8), turned to 90 degrees
- moved Q3 0.25 mm to (97.8, 78.5), turned to 90 degrees
Connections:
- Q1 pad 2: Net-(Q1-Pad2) -> +5V
- Q1 pad 3: +5V -> Net-(Q1-Pad3)
- Q2 pad 2: Net-(Q2-Pad2) -> +5V
- Q2 pad 3: +5V -> Net-(Q2-Pad3)
- Q3 pad 2: Net-(Q3-Pad2) -> +5V
- Q3 pad 3: +5V -> Net-(Q3-Pad3)
- U3 pad 3: Net-(Q1-Pad2) -> Net-(Q1-Pad3)
- U3 pad 8: Net-(Q1-Pad2) -> Net-(Q1-Pad3)
- U4 pad 3: Net-(Q2-Pad2) -> Net-(Q2-Pad3)
- U4 pad 8: Net-(Q2-Pad2) -> Net-(Q2-Pad3)
- U5 pad 3: Net-(Q3-Pad2) -> Net-(Q3-Pad3)
- U5 pad 8: Net-(Q3-Pad2) -> Net-(Q3-Pad3)
Routing:
- net /SEG_SEL_0: track 61.3 -> 53.3 mm
- net /SEG_SEL_1: track 25.9 -> 19.5 mm
- net Net-(Q1-Pad2): track 4.06 -> 0.00 mm
- net Net-(Q1-Pad3): track 0.00 -> 3.76 mm
- net Net-(Q3-Pad1): track 5.96 -> 2.30 mm
- net Net-(Q2-Pad2): track 3.56 -> 0.00 mm
- net Net-(Q3-Pad3): track 0.00 -> 3.32 mm
- net Net-(Q3-Pad2): track 3.27 -> 0.00 mm
- net Net-(Q2-Pad3): track 0.00 -> 3.26 mm
- net GND: track 63.1 -> 65.9 mm, vias 70 -> 71
- net +5V: track 167.6 -> 170.2 mm, vias 9 -> 10
- net TX_F: track 51.7 -> 53.6 mm, vias 2 -> 0
- net Net-(Q1-Pad1): track 3.89 -> 2.52 mm
- net RX_F: track 48.3 -> 47.0 mm, vias 2 -> 0
- net Net-(Q2-Pad1): track 3.89 -> 2.77 mm
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Other:
- board text added: "v0.2.2, Jan 2021"
- board text removed: "v0.2.0, Dec 2020"

Commit message: v0.2.3 PCB Updated, board step file generated
Parts:
- U3, U4, U5: footprint lsd100bag-101-20:lsd100bag-101-20 -> lsd100bag-101-20:lsd100bag-101
- moved U5 1.70 mm to (100.2, 90.0)
- moved U3 1.70 mm to (148.8, 90.0)
Routing:
- net TX_F: track 53.6 -> 46.0 mm
- net /SEG_A: track 64.5 -> 60.2 mm
- net /SEG_F: track 65.7 -> 62.3 mm
- net /SEG_B: track 63.2 -> 60.1 mm
- net +3V3: track 61.5 -> 58.6 mm
- net /SEG_D: track 65.7 -> 63.0 mm
- net /SEG_E: track 66.4 -> 64.0 mm
- net /SEG_C: track 67.8 -> 65.4 mm
- net /SEG_RDP: track 66.7 -> 64.4 mm
- net /SEG_G: track 65.0 -> 63.4 mm
- net GND: track 65.9 -> 64.3 mm
- net Net-(Q3-Pad3): track 3.32 -> 4.76 mm
- net Net-(Q1-Pad3): track 3.76 -> 4.91 mm
Other:
- rule pad_to_mask_clearance: 0.05 -> 0
- board text added: "v0.2.3, Jan 2021"
- board text removed: "v0.2.2, Jan 2021"

Commit message: v0.2.4 PCB Updated
Parts:
- moved SW1 1.25 mm to (101.2, 120.0)
- moved SW10 1.25 mm to (141.2, 140.0)
- moved SW11 1.25 mm to (141.2, 160.0)
- moved SW12 1.25 mm to (141.2, 180.0)
- moved SW2 1.25 mm to (101.2, 140.0)
- moved SW3 1.25 mm to (101.2, 160.0)
- moved SW4 1.25 mm to (101.2, 180.0)
- moved SW5 1.25 mm to (121.2, 120.0)
- moved SW6 1.25 mm to (121.2, 140.0)
- moved SW7 1.25 mm to (121.2, 160.0)
- moved SW8 1.25 mm to (121.2, 180.0)
- moved SW9 1.25 mm to (141.2, 120.0)
- moved H1 0.50 mm to (86.5, 67.5)
- moved H2 0.50 mm to (86.5, 111.0)
- moved H3 0.50 mm to (86.5, 190.0)
Routing:
- net MOSI: track 184.3 -> 189.4 mm
- net /ROW_3: track 143.9 -> 145.8 mm
- net RESET: track 81.0 -> 79.5 mm
- net SCK: track 47.3 -> 46.1 mm
- net MISO: track 230.9 -> 232.0 mm
- net P_LED: track 51.4 -> 50.4 mm
- net /COL_2: track 137.8 -> 136.8 mm
- net /ROW_2: track 123.1 -> 123.6 mm
Other:
- board size 81 x 128.5 mm -> 80.5 x 128.5 mm
- board text added: "v0.2.4, Jan 2021"
- board text removed: "v0.2.3, Jan 2021"
